File: m0110a_qmk.kicad_pcb (KiCad board)
At the start: 2 copper layers, 179 parts, among them J1 AVR-ISP-6, J2 USB_B_Mini, U1 ATmega32A-PU, Y1 16Mhz

Commit message: finished pcb layout
Parts:
- removed D68: D_Small, Diodes_THT:D_DO-35_SOD27_P7.62mm_Horizontal
- removed MX66: MX-NoLED, Alps_Only:ALPS-1U
- D10, D11, D12, D13, D14, D15, D16, D17, D18, D19, D20, D21, D22, D23, D24, D25, D26, D27, D28, D29, D3, D30, D31, D32, D33, D34, D35, D36, D37, D38, D39, D4, D40, D41, D42, D43, D44, D45, D46, D47, D48, D49, D5, D50, D51, D52, D53, D54, D55, D56, D57, D58, D59, D6, D60, D61, D62, D63, D64, D65, D66, D67, D69, D7, D70, D71, D72, D73, D74, D75, D76, D77, D78, D79, D8, D80, D81, D9: moved to B.Cu
- F1: footprint Alps_Only:ALPS-1U -> Fuse_Holders_and_Fuses:Fuse_TE5_Littlefuse-395Series
- J1: footprint Alps_Only:ALPS-1U -> Pin_Headers:Pin_Header_Angled_2x03_Pitch2.54mm
- J2: footprint Alps_Only:ALPS-1U -> random-keyboard-parts:Molex-0548190519
- MX1, MX10, MX11, MX12, MX13, MX14, MX15, MX16, MX17, MX18, MX19, MX2, MX20, MX21, MX22, MX23, MX24, MX25, MX26, MX27, MX28, MX29, MX3, MX30, MX31, MX32, MX33, MX34, MX35, MX36, MX37, MX38, MX39, MX4, MX40, MX41, MX42, MX43, MX44, MX45, MX46, MX47, MX48, MX49, MX5, MX50, MX51, MX52, MX53, MX54, MX55, MX56, MX57, MX58, MX59, MX6, MX60, MX61, MX62, MX63, MX64, MX65, MX67, MX68, MX69, MX7, MX70, MX71, MX72, MX73, MX74, MX75, MX76, MX77, MX78, MX79, MX8, MX80, MX9: footprint Alps_Only:ALPS-1U -> Alps_Only:ALPS-SKCC
- moved MX18 366.4 mm to (381.9, 85.9)
- moved MX79 355.8 mm to (383.4, 150.7), turned to 90 degrees
- moved D70 339.7 mm to (353.3, 146.3), turned to 90 degrees
- moved MX78 331.8 mm to (362.8, 162.1)
- moved MX35 304.9 mm to (381.9, 104.9)
- moved MX69 303.3 mm to (362.8, 143.0)
- moved MX68 301.6 mm to (343.8, 143.0)
- moved MX33 291.3 mm to (343.8, 104.9)
- moved MX49 284.8 mm to (324.7, 124.0)
- moved MX34 262.4 mm to (362.8, 104.9)
- moved MX50 259.5 mm to (343.8, 124.0)
- moved MX77 257.2 mm to (334.3, 162.1)
- moved MX75 255.0 mm to (275.7, 162.1)
- moved MX67 251.1 mm to (324.7, 143.0)
- moved MX1 250.1 mm to (37.0, 85.9)
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Connections:
- D16 pad 1: row0 -> row4
- MX14 pad 1: col13 -> col8
- MX73 pad 1: col7 -> col9
- MX74 pad 1: col8 -> col10
- MX75 pad 1: col9 -> col11
- MX76 pad 1: col10 -> col12
- U1 pad 1: col3 -> row0
- U1 pad 14: col16 -> Net-(U1-Pad14)
- U1 pad 15: col17 -> Net-(U1-Pad15)
- U1 pad 19: Net-(U1-Pad19) -> row4
- U1 pad 2: col4 -> row1
- U1 pad 20: Net-(U1-Pad20) -> col5
- U1 pad 21: Net-(U1-Pad21) -> col0
- U1 pad 22: col8 -> col1
- U1 pad 23: col9 -> col2
- U1 pad 24: col10 -> col3
- U1 pad 25: col11 -> col4
- U1 pad 26: col12 -> Net-(U1-Pad26)
- U1 pad 27: col13 -> Net-(U1-Pad27)
- U1 pad 28: col14 -> col7
- U1 pad 29: col15 -> col8
- U1 pad 3: col5 -> row2
- U1 pad 33: col2 -> col9
- U1 pad 34: col1 -> col10
- U1 pad 35: col0 -> col11
- U1 pad 36: row4 -> col12
- U1 pad 37: row3 -> col17
- U1 pad 38: row2 -> col16
- U1 pad 39: row1 -> col15
- U1 pad 4: col6 -> row3
- U1 pad 40: row0 -> col14
- U1 pad 5: col7 -> col6
Routing:
- net GND: track 0.00 -> 503.5 mm
- net row4: track 0.00 -> 440.9 mm
- net row0: track 0.00 -> 434.0 mm
- net row1: track 0.00 -> 400.7 mm
- net +5V: track 0.00 -> 389.2 mm, vias 0 -> 1
- net row2: track 0.00 -> 378.6 mm
- net row3: track 0.00 -> 326.0 mm
- net reset: track 0.00 -> 323.3 mm, vias 0 -> 3
- net col17: track 0.00 -> 294.8 mm, vias 0 -> 1
- net col16: track 0.00 -> 267.5 mm, vias 0 -> 1
- net col8: track 0.00 -> 247.2 mm, vias 0 -> 1
- net col15: track 0.00 -> 245.1 mm, vias 0 -> 1
- net col14: track 0.00 -> 235.6 mm, vias 0 -> 1
- net col12: track 0.00 -> 213.6 mm, vias 0 -> 1
- net SCK: track 0.00 -> 202.2 mm, vias 0 -> 2
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Other:
- net class Power added: clearance 0.2, trace_width 0.5, via_dia 0.8, via_drill 0.4

Commit message: finish pcb
Routing:
- net D-: track 124.2 -> 126.3 mm
- net MOSI: track 201.7 -> 202.6 mm
- net reset: track 323.3 -> 324.0 mm
Other:
- board outline added: 380 x 137.9 mm

Commit message: fixed USB port orientation
Parts:
- J2: moved to B.Cu
- moved C3 17.8 mm to (91.3, 72.8), turned to 180 degrees
- moved F1 17.0 mm to (92.7, 66.4), turned to 180 degrees
- moved R5 9.40 mm to (82.5, 64.4)
- moved R3 8.77 mm to (78.4, 64.4)
- moved R2 8.13 mm to (74.2, 64.4)
Routing:
- net GND: track 503.5 -> 483.3 mm
- net D-: track 126.3 -> 135.3 mm
- net Net-(D2-Pad1): track 30.2 -> 21.4 mm
- net D+: track 129.1 -> 137.5 mm
- net Net-(J2-Pad6): track 0.00 -> 7.30 mm
- net row4: track 440.9 -> 447.7 mm
- net +5V: track 389.2 -> 393.0 mm
- net Net-(D1-Pad1): track 33.1 -> 29.4 mm
- net Net-(J2-Pad4): track 0.00 -> 0.84 mm
- net VCC: track 7.01 -> 6.19 mm

Commit message: flipped diodes and added groundplanes
Parts:
- D10, D11, D12, D13, D14, D15, D16, D17, D18, D19, D20, D21, D22, D23, D24, D25, D26, D27, D28, D29, D3, D30, D31, D32, D33, D34, D35, D36, D37, D38, D39, D4, D40, D41, D42, D43, D44, D45, D46, D47, D48, D49, D5, D50, D51, D52, D53, D54, D55, D56, D57, D58, D59, D6, D60, D61, D62, D63, D64, D65, D66, D67, D69, D7, D70, D71, D72, D73, D74, D75, D76, D77, D78, D79, D8, D80, D81, D9: moved to F.Cu
Routing:
- net Net-(J2-Pad6): track 7.30 -> 0.00 mm
- net D-: track 135.3 -> 136.2 mm
- net GND: vias 0 -> 2
- added copper zone on B.Cu, net GND
- added copper zone on F.Cu, net GND

Commit message: changed footprints
Parts:
- added G***: LOGO, custom_parts:apple_x_elmo, B.Cu at (106.7, 156.7)
- MX1, MX10, MX11, MX12, MX13, MX14, MX15, MX16, MX17, MX18, MX19, MX2, MX20, MX21, MX22, MX23, MX24, MX25, MX26, MX27, MX28, MX29, MX3, MX30, MX31, MX32, MX33, MX34, MX35, MX36, MX37, MX38, MX39, MX4, MX40, MX41, MX42, MX43, MX44, MX45, MX46, MX47, MX48, MX49, MX5, MX50, MX51, MX52, MX53, MX54, MX55, MX56, MX57, MX58, MX59, MX6, MX60, MX61, MX62, MX63, MX64, MX65, MX67, MX68, MX69, MX7, MX70, MX71, MX72, MX73, MX74, MX75, MX76, MX77, MX78, MX79, MX8, MX80, MX9: footprint Alps_Only:ALPS-SKCC -> custom_parts:alps_skcc
Other:
- board text added: "M0110a QMK PCB v0.1"

Commit message: small update
Parts:
- added G***: LOGO, custom_parts:oshw, B.Cu at (93.5, 169.7)
