File: m0110a_qmk.kicad_pcb (KiCad board)
At the start: 2 copper layers, 380 x 137.9 mm, 179 parts, among them J1 USB_B_Mini, J2 AVR-ISP-6, U1 ATmega32A-PU, Y1 Resonator

Commit message: change JST connector size
Parts:
- removed Y1: Resonator, Crystal:Resonator-3Pin_W7.0mm_H2.5mm
- added C4: 22p, Capacitor_THT:C_Disc_D6.0mm_W2.5mm_P5.00mm, F.Cu at (160.3, 155.6)
- added C5: 22p, Capacitor_THT:C_Disc_D6.0mm_W2.5mm_P5.00mm, F.Cu at (175.8, 155.6)
- added XTAL1: Crystal, Crystal:Crystal_HC49-4H_Vertical, F.Cu at (165.6, 153.8)
- J1: value USB_B_Mini -> Conn_01x04; footprint random-keyboard-parts:Molex-0548190519 -> Connector_JST:JST_PH_S4B-PH-K_1x04_P2.00mm_Horizontal
- moved J1 33.4 mm to (114.0, 69.0), turned to 180 degrees
- moved C3 8.89 mm to (179.3, 154.6), turned to 90 degrees
- moved F1 5.08 mm to (87.6, 66.4), turned to 0 degrees
- moved R5 0.46 mm to (56.9, 72.8)
Connections:
- J1 pad 1: VCC -> GND
- J1 pad 4: Net-(J1-Pad4) -> VCC
Routing:
- net GND: track 89.0 -> 0.06 mm
- net Net-(D1-Pad1): track 18.0 -> 51.1 mm
- net Net-(D2-Pad1): track 32.5 -> 60.2 mm
- net VCC: track 6.19 -> 16.4 mm
- net Net-(C5-Pad1): track 4.56 -> 13.1 mm
- net Net-(C4-Pad1): track 4.59 -> 11.9 mm
- net +5V: track 371.3 -> 374.7 mm

Commit message: update
Parts:
- moved G*** 8.40 mm to (85.6, 172.6)
- moved G*** 5.08 mm to (110.4, 172.2)
Other:
- board text added: "github.com/kb-elmo/m0110a_usb elmo.space"
