File: m0110a_qmk.sch (KiCad schematic (older format))
At the start: 18 parts, among them J1 AVR-ISP-6, J2 USB_B_Mini, Y1 16Mhz

Commit message: some changes to the controller circuit
Parts:
- added D3: LED, symbol Device:LED
- added R5: 1.5k, symbol Device:R
- renumbered R1 to R4
Connections:
- wire segments 60 -> 61
Other:
- moved on the sheet: D1, D2, F1, J2, R1, R2, R3

Commit message: finished circuit schema
Parts:
- added D10, D11, D12, D13, D14, D15, D16, D17, D18, D19, D20, D21, D4, D5, D6, D7, D8, D9, D? (x61): D_Small, symbol Device:D_Small
- added MX1: ESC, symbol MX_Alps_Hybrid:MX-NoLED
- added MX10: 9, symbol MX_Alps_Hybrid:MX-NoLED
- added MX11: 0, symbol MX_Alps_Hybrid:MX-NoLED
- added MX12: minus, symbol MX_Alps_Hybrid:MX-NoLED
- added MX13: plus, symbol MX_Alps_Hybrid:MX-NoLED
- added MX14: bkspc, symbol MX_Alps_Hybrid:MX-NoLED
- added MX15: clear, symbol MX_Alps_Hybrid:MX-NoLED
- added MX16: num-eq, symbol MX_Alps_Hybrid:MX-NoLED
- added MX17: num-div, symbol MX_Alps_Hybrid:MX-NoLED
- added MX18: num-mul, symbol MX_Alps_Hybrid:MX-NoLED
- added MX2: 1, symbol MX_Alps_Hybrid:MX-NoLED
- added MX3: 2, symbol MX_Alps_Hybrid:MX-NoLED
- added MX4: 3, symbol MX_Alps_Hybrid:MX-NoLED
- added MX5: 4, symbol MX_Alps_Hybrid:MX-NoLED
- added MX6: 5, symbol MX_Alps_Hybrid:MX-NoLED
- added MX7: 6, symbol MX_Alps_Hybrid:MX-NoLED
- added MX8: 7, symbol MX_Alps_Hybrid:MX-NoLED
- added MX9: 8, symbol MX_Alps_Hybrid:MX-NoLED
- added MX? (x61): MX-NoLED, symbol MX_Alps_Hybrid:MX-NoLED
Connections:
- net col3: now reaches U?.1 (PB0)
- net col3: now also MX4.1 (COL), MX?.1 (COL), MX?.1 (COL), MX?.1 (COL)
- net col16: now reaches U?.14 (PD0)
- net col16: now also MX17.1 (COL), MX?.1 (COL), MX?.1 (COL), MX?.1 (COL), MX?.1 (COL)
- net col17: now reaches U?.15 (PD1)
- net col17: now also MX18.1 (COL), MX?.1 (COL), MX?.1 (COL), MX?.1 (COL)
- net col4: now reaches U?.2 (PB1)
- net col4: now also MX5.1 (COL), MX?.1 (COL), MX?.1 (COL), MX?.1 (COL), MX?.1 (COL)
- net col8: now reaches U?.22 (PC0)
- net col8: now also MX9.1 (COL), MX?.1 (COL), MX?.1 (COL), MX?.1 (COL), MX?.1 (COL)
- net col9: now reaches U?.23 (PC1)
- net col9: now also MX10.1 (COL), MX?.1 (COL), MX?.1 (COL), MX?.1 (COL), MX?.1 (COL)
- net col10: now reaches U?.24 (PC2)
- net col10: now also MX11.1 (COL), MX?.1 (COL), MX?.1 (COL), MX?.1 (COL), MX?.1 (COL)
- net col11: now reaches U?.25 (PC3)
- net col11: now also MX12.1 (COL), MX?.1 (COL), MX?.1 (COL), MX?.1 (COL)
- net col12: now reaches U?.26 (PC4)
- net col12: now also MX13.1 (COL), MX?.1 (COL), MX?.1 (COL), MX?.1 (COL)
- net col13: now reaches U?.27 (PC5)
- net col13: now also MX14.1 (COL), MX?.1 (COL)
- net col14: now reaches U?.28 (PC6)
- net col14: now also MX15.1 (COL), MX?.1 (COL), MX?.1 (COL), MX?.1 (COL), MX?.1 (COL)
- net col15: now reaches U?.29 (PC7)
- net col15: now also MX16.1 (COL), MX?.1 (COL), MX?.1 (COL), MX?.1 (COL)
- net col5: now reaches U?.3 (PB2)
- net col5: now also MX6.1 (COL), MX?.1 (COL), MX?.1 (COL), MX?.1 (COL)
- net col2: now reaches U?.33 (PA7)
- net col2: now also MX3.1 (COL), MX?.1 (COL), MX?.1 (COL), MX?.1 (COL)
- net col1: now reaches U?.34 (PA6)
- net col1: now also MX2.1 (COL), MX?.1 (COL), MX?.1 (COL), MX?.1 (COL), MX?.1 (COL)
- net col0: now reaches U?.35 (PA5)
- net col0: now also MX1.1 (COL), MX?.1 (COL), MX?.1 (COL), MX?.1 (COL), MX?.1 (COL)
- net row4: now reaches U?.36 (PA4)
- net row4: now also D?.1 (K), D?.1 (K), D?.1 (K), D?.1 (K), D?.1 (K), D?.1 (K), D?.1 (K), D?.1 (K), D?.1 (K), D?.1 (K)
- net row3: now reaches U?.37 (PA3)
- net row3: now also D?.1 (K), D?.1 (K), D?.1 (K), D?.1 (K), D?.1 (K), D?.1 (K), D?.1 (K), D?.1 (K), D?.1 (K), D?.1 (K), D?.1 (K), D?.1 (K), D?.1 (K), D?.1 (K), D?.1 (K), D?.1 (K), D?.1 (K)
- net row2: now reaches U?.38 (PA2)
- net row2: now also D?.1 (K), D?.1 (K), D?.1 (K), D?.1 (K), D?.1 (K), D?.1 (K), D?.1 (K), D?.1 (K), D?.1 (K), D?.1 (K), D?.1 (K), D?.1 (K), D?.1 (K), D?.1 (K), D?.1 (K), D?.1 (K), D?.1 (K)
- net row1: now reaches U?.39 (PA1)
- net row1: now also D?.1 (K), D?.1 (K), D?.1 (K), D?.1 (K), D?.1 (K), D?.1 (K), D?.1 (K), D?.1 (K), D?.1 (K), D?.1 (K), D?.1 (K), D?.1 (K), D?.1 (K), D?.1 (K), D?.1 (K), D?.1 (K), D?.1 (K)
- net col6: now reaches U?.4 (PB3)
- net col6: now also MX7.1 (COL), MX?.1 (COL), MX?.1 (COL), MX?.1 (COL)
- net row0: now reaches U?.40 (PA0)
- net row0: now also D10.1 (K), D11.1 (K), D12.1 (K), D13.1 (K), D14.1 (K), D15.1 (K), D16.1 (K), D17.1 (K), D18.1 (K), D19.1 (K), D20.1 (K), D21.1 (K), D4.1 (K), D5.1 (K), D6.1 (K), D7.1 (K), D8.1 (K), D9.1 (K)
- net col7: now reaches U?.5 (PB4)
- net col7: now also MX8.1 (COL), MX?.1 (COL), MX?.1 (COL), MX?.1 (COL), MX?.1 (COL)
- new net: D4.2 (A), MX1.2 (ROW)
- new net: D5.2 (A), MX2.2 (ROW)
- new net: D6.2 (A), MX3.2 (ROW)
- new net: D7.2 (A), MX4.2 (ROW)
- new net: D8.2 (A), MX5.2 (ROW)
- new net: D9.2 (A), MX6.2 (ROW)
- new net: D10.2 (A), MX7.2 (ROW)
- new net: D11.2 (A), MX8.2 (ROW)
- new net: D12.2 (A), MX9.2 (ROW)
- new net: D13.2 (A), MX10.2 (ROW)
- new net: D14.2 (A), MX11.2 (ROW)
- new net: D15.2 (A), MX12.2 (ROW)
- new net: D16.2 (A), MX13.2 (ROW)
- new net: D17.2 (A), MX14.2 (ROW)
- new net: D18.2 (A), MX15.2 (ROW)
- new net: D19.2 (A), MX16.2 (ROW)
- new net: D20.2 (A), MX17.2 (ROW)
- new net: D21.2 (A), MX18.2 (ROW)
- new net: D?.2 (A), MX?.2 (ROW) (x61)
Other:
- moved on the sheet: Boot1, C1, C2, C3, C4, C5, D1, D2, D3, F1, J1, J2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

Commit message: finish footprint matching
Parts:
- added MX80: MX-NoLED, Alps_Only:ALPS-1U, symbol MX_Alps_Hybrid:MX-NoLED
- Boot1, Reset1: footprint (none) -> Buttons_Switches_THT:SW_PUSH_6mm
- C1, C2: footprint (none) -> Capacitors_THT:C_Disc_D6.0mm_W2.5mm_P5.00mm
- C3: footprint (none) -> Capacitors_THT:CP_Radial_D5.0mm_P2.50mm
- C4, C5: footprint (none) -> Capacitors_THT:C_Disc_D3.0mm_W2.0mm_P2.50mm
- D1, D2: footprint (none) -> Diodes_THT:D_DO-35_SOD27_P7.62mm_Horizontal
- D10: renamed from D11; footprint (none) -> Diodes_THT:D_DO-35_SOD27_P7.62mm_Horizontal
- D11: renamed from D12; footprint (none) -> Diodes_THT:D_DO-35_SOD27_P7.62mm_Horizontal
- D12: renamed from D13; footprint (none) -> Diodes_THT:D_DO-35_SOD27_P7.62mm_Horizontal
- D13: renamed from D14; footprint (none) -> Diodes_THT:D_DO-35_SOD27_P7.62mm_Horizontal
- D14: renamed from D15; footprint (none) -> Diodes_THT:D_DO-35_SOD27_P7.62mm_Horizontal
- D15: renamed from D16; footprint (none) -> Diodes_THT:D_DO-35_SOD27_P7.62mm_Horizontal
- D16: renamed from D17; footprint (none) -> Diodes_THT:D_DO-35_SOD27_P7.62mm_Horizontal
- D17: renamed from D18; footprint (none) -> Diodes_THT:D_DO-35_SOD27_P7.62mm_Horizontal
- D18: renamed from D19; footprint (none) -> Diodes_THT:D_DO-35_SOD27_P7.62mm_Horizontal
- D19: renamed from D20; footprint (none) -> Diodes_THT:D_DO-35_SOD27_P7.62mm_Horizontal
- D20: renamed from D21; footprint (none) -> Diodes_THT:D_DO-35_SOD27_P7.62mm_Horizontal
- D21, D22, D23, D24, D25, D26, D27, D28, D29, D30, D31, D32, D33, D34, D35, D36, D37, D38, D39, D40, D41, D42, D43, D44, D45, D46, D47, D48, D49, D50, D51, D52, D53, D54, D55, D56, D57, D58, D59, D60, D61, D62, D63, D64, D65, D66, D67, D68, D69, D70, D71, D72, D73, D74, D75, D76, D77, D78, D79, D80, D81: renamed from D?; footprint (none) -> Diodes_THT:D_DO-35_SOD27_P7.62mm_Horizontal
- D3: renamed from D4; footprint (none) -> Diodes_THT:D_DO-35_SOD27_P7.62mm_Horizontal
- D4: renamed from D5; footprint (none) -> Diodes_THT:D_DO-35_SOD27_P7.62mm_Horizontal
- D5: renamed from D6; footprint (none) -> Diodes_THT:D_DO-35_SOD27_P7.62mm_Horizontal
- D6: renamed from D7; footprint (none) -> Diodes_THT:D_DO-35_SOD27_P7.62mm_Horizontal
- D7: renamed from D8; footprint (none) -> Diodes_THT:D_DO-35_SOD27_P7.62mm_Horizontal
- D8: renamed from D9; footprint (none) -> Diodes_THT:D_DO-35_SOD27_P7.62mm_Horizontal
- D82: renamed from D3; footprint (none) -> LEDs:LED_D3.0mm
- D9: renamed from D10; footprint (none) -> Diodes_THT:D_DO-35_SOD27_P7.62mm_Horizontal
- F1, J1, J2, MX1, MX10, MX11, MX12, MX13, MX14, MX15, MX16, MX17, MX18, MX2, MX3, MX4, MX5, MX6, MX7, MX8, MX9: footprint (none) -> Alps_Only:ALPS-1U
- MX19, MX20, MX21, MX22, MX23, MX24, MX25, MX26, MX27, MX28, MX29, MX30, MX31, MX32, MX33, MX34, MX35, MX36, MX37, MX38, MX39, MX40, MX41, MX42, MX43, MX44, MX45, MX46, MX47, MX48, MX49, MX50, MX51, MX52, MX53, MX54, MX55, MX56, MX57, MX58, MX59, MX60, MX61, MX62, MX63, MX64, MX65, MX66, MX67, MX68, MX69, MX70, MX71, MX72, MX73, MX74, MX75, MX76, MX77, MX78, MX79: renamed from MX?; footprint (none) -> Alps_Only:ALPS-1U
- R1: renamed from R4; footprint (none) -> Resistors_THT:R_Axial_DIN0207_L6.3mm_D2.5mm_P10.16mm_Horizontal
- R2: renamed from R1; footprint (none) -> Resistors_THT:R_Axial_DIN0207_L6.3mm_D2.5mm_P10.16mm_Horizontal
- R3: renamed from R2; footprint (none) -> Resistors_THT:R_Axial_DIN0207_L6.3mm_D2.5mm_P10.16mm_Horizontal
- R4: renamed from R5; footprint (none) -> Resistors_THT:R_Axial_DIN0207_L6.3mm_D2.5mm_P10.16mm_Horizontal
- R5: renamed from R3; footprint (none) -> Resistors_THT:R_Axial_DIN0207_L6.3mm_D2.5mm_P10.16mm_Horizontal
- U1: renamed from U?; footprint Package_DIP:DIP-40_W15.24mm -> Housings_DIP:DIP-40_W15.24mm
- Y1: footprint (none) -> Crystals:Crystal_HC49-U_Vertical

Commit message: finished pcb layout
Parts:
- removed D68: D_Small, Diodes_THT:D_DO-35_SOD27_P7.62mm_Horizontal, symbol Device:D_Small
- removed MX66: MX-NoLED, Alps_Only:ALPS-1U, symbol MX_Alps_Hybrid:MX-NoLED
- F1: footprint Alps_Only:ALPS-1U -> Fuse_Holders_and_Fuses:Fuse_TE5_Littlefuse-395Series
- J1: footprint Alps_Only:ALPS-1U -> Pin_Headers:Pin_Header_Angled_2x03_Pitch2.54mm
- J2: footprint Alps_Only:ALPS-1U -> random-keyboard-parts:Molex-0548190519
- MX1, MX10, MX11, MX12, MX13, MX14, MX15, MX16, MX17, MX18, MX19, MX2, MX20, MX21, MX22, MX23, MX24, MX25, MX26, MX27, MX28, MX29, MX3, MX30, MX31, MX32, MX33, MX34, MX35, MX36, MX37, MX38, MX39, MX4, MX40, MX41, MX42, MX43, MX44, MX45, MX46, MX47, MX48, MX49, MX5, MX50, MX51, MX52, MX53, MX54, MX55, MX56, MX57, MX58, MX59, MX6, MX60, MX61, MX62, MX63, MX64, MX65, MX67, MX68, MX69, MX7, MX70, MX71, MX72, MX73, MX74, MX75, MX76, MX77, MX78, MX79, MX8, MX80, MX9: footprint Alps_Only:ALPS-1U -> Alps_Only:ALPS-SKCC
Connections:
- net col0: now also U1.21 (PD7); no longer U1.35 (PA5)
- net col1: now also U1.22 (PC0); no longer U1.34 (PA6)
- net col10: now also MX74.1 (COL), U1.34 (PA6); no longer MX76.1 (COL), U1.24 (PC2)
- net col11: now also MX75.1 (COL), U1.35 (PA5); no longer U1.25 (PC3)
- net col12: now also MX76.1 (COL), U1.36 (PA4); no longer U1.26 (PC4)
- net col14: now also U1.40 (PA0); no longer U1.28 (PC6)
- net col15: now also U1.39 (PA1); no longer U1.29 (PC7)
- net col16: now also U1.38 (PA2); no longer U1.14 (PD0)
- net col17: now also U1.37 (PA3); no longer U1.15 (PD1)
- net col2: now also U1.23 (PC1); no longer U1.33 (PA7)
- net col3: now also U1.24 (PC2); no longer U1.1 (PB0)
- net col4: now also U1.25 (PC3); no longer U1.2 (PB1)
- net col5: now also U1.20 (PD6); no longer U1.3 (PB2)
- net col6: now also U1.5 (PB4); no longer U1.4 (PB3)
- net col7: now also U1.28 (PC6); no longer MX73.1 (COL), U1.5 (PB4)
- net col8: now also MX14.1 (COL), U1.29 (PC7); no longer MX74.1 (COL), U1.22 (PC0)
- net col9: now also MX73.1 (COL), U1.33 (PA7); no longer MX75.1 (COL), U1.23 (PC1)
- net row0: now also U1.1 (PB0); no longer D16.1 (K), U1.40 (PA0)
- net row1: now also U1.2 (PB1); no longer U1.39 (PA1)
- net row2: now also U1.3 (PB2); no longer U1.38 (PA2)
- net row3: now also U1.4 (PB3); no longer U1.37 (PA3)
- net row4: now also D16.1 (K), U1.19 (PD5); no longer U1.36 (PA4)
- net col13: no longer names the net of U1.27 (PC5)
- net col13: no longer MX14.1 (COL)
Other:
- moved on the sheet: D16, D75, D76, D77, D78, MX14, MX73, MX74, MX75, MX76

Commit message: changed footprints
Parts:
- MX1, MX10, MX11, MX12, MX13, MX14, MX15, MX16, MX17, MX18, MX19, MX2, MX20, MX21, MX22, MX23, MX24, MX25, MX26, MX27, MX28, MX29, MX3, MX30, MX31, MX32, MX33, MX34, MX35, MX36, MX37, MX38, MX39, MX4, MX40, MX41, MX42, MX43, MX44, MX45, MX46, MX47, MX48, MX49, MX5, MX50, MX51, MX52, MX53, MX54, MX55, MX56, MX57, MX58, MX59, MX6, MX60, MX61, MX62, MX63, MX64, MX65, MX67, MX68, MX69, MX7, MX70, MX71, MX72, MX73, MX74, MX75, MX76, MX77, MX78, MX79, MX8, MX80, MX9: footprint Alps_Only:ALPS-SKCC -> custom_parts:alps_skcc

Commit message: fixes for newer keycad versions
fixed pathes for 3d parts
Parts:
- Boot1, Reset1: footprint Buttons_Switches_THT:SW_PUSH_6mm -> Button_Switch_THT:SW_PUSH_6mm
- C1, C2: footprint Capacitors_THT:C_Disc_D6.0mm_W2.5mm_P5.00mm -> Capacitor_THT:C_Disc_D6.0mm_W2.5mm_P5.00mm
- C3: footprint Capacitors_THT:CP_Radial_D5.0mm_P2.50mm -> Capacitor_THT:CP_Radial_D5.0mm_P2.50mm
- C4, C5: footprint Capacitors_THT:C_Disc_D3.0mm_W2.0mm_P2.50mm -> Capacitor_THT:C_Disc_D3.0mm_W2.0mm_P2.50mm
- D1, D10, D11, D12, D13, D14, D15, D16, D17, D18, D19, D2, D20, D21, D22, D23, D24, D25, D26, D27, D28, D29, D3, D30, D31, D32, D33, D34, D35, D36, D37, D38, D39, D4, D40, D41, D42, D43, D44, D45, D46, D47, D48, D49, D5, D50, D51, D52, D53, D54, D55, D56, D57, D58, D59, D6, D60, D61, D62, D63, D64, D65, D66, D67, D69, D7, D70, D71, D72, D73, D74, D75, D76, D77, D78, D79, D8, D80, D81, D9: footprint Diodes_THT:D_DO-35_SOD27_P7.62mm_Horizontal -> Diode_THT:D_DO-35_SOD27_P7.62mm_Horizontal
- D82: footprint LEDs:LED_D3.0mm -> LED_THT:LED_D3.0mm
- F1: footprint Fuse_Holders_and_Fuses:Fuse_TE5_Littlefuse-395Series -> Fuse:Fuse_Littelfuse_395Series
- J1: footprint Pin_Headers:Pin_Header_Angled_2x03_Pitch2.54mm -> Connector_PinHeader_2.54mm:PinHeader_2x03_P2.54mm_Horizontal
- R1, R2, R3, R4, R5: footprint Resistors_THT:R_Axial_DIN0207_L6.3mm_D2.5mm_P10.16mm_Horizontal -> Resistor_THT:R_Axial_DIN0207_L6.3mm_D2.5mm_P10.16mm_Horizontal
- U1: footprint Housings_DIP:DIP-40_W15.24mm -> Package_DIP:DIP-40_W15.24mm_Socket
- Y1: footprint Crystals:Crystal_HC49-U_Vertical -> Crystal:Crystal_HC49-4H_Vertical

Commit message: fix some mistakes
Parts:
- F1: footprint Fuse:Fuse_Littelfuse_395Series -> custom_parts:Fuse_Littelfuse_395Series
Connections:
- net col14: now also MX16.1 (COL), MX33.1 (COL), MX50.1 (COL), MX68.1 (COL), U1.38 (PA2); no longer MX15.1 (COL), MX32.1 (COL), MX49.1 (COL), MX67.1 (COL), MX77.1 (COL), U1.40 (PA0)
- net col15: now also MX17.1 (COL), MX34.1 (COL), MX51.1 (COL), MX69.1 (COL), MX78.1 (COL); no longer MX16.1 (COL), MX33.1 (COL), MX50.1 (COL), MX68.1 (COL)
- net col16: now also MX18.1 (COL), MX35.1 (COL), MX52.1 (COL), MX79.1 (COL), U1.40 (PA0); no longer MX17.1 (COL), MX34.1 (COL), MX51.1 (COL), MX69.1 (COL), MX78.1 (COL), U1.38 (PA2)
- net at D2.1 (K), J2.2 (D-), R3.1: now also R5.2
- net at D1.1 (K), J2.3 (D+), R2.1: no longer R5.2
- removed net col17: MX18.1 (COL), MX35.1 (COL), MX52.1 (COL), MX79.1 (COL), U1.37 (PA3)
- new net col13: MX15.1 (COL), MX32.1 (COL), MX49.1 (COL), MX67.1 (COL), MX77.1 (COL), U1.37 (PA3)
Other:
- moved on the sheet: Boot1, C1, C2, C3, C4, C5, D1, D10, D11, D12, D13, D14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

Commit message: rev1
Parts:
- removed C1, C2: 22p, Capacitor_THT:C_Disc_D6.0mm_W2.5mm_P5.00mm, symbol Device:C
- removed MX80: MX-NoLED, custom_parts:alps_skcc, symbol MX_Alps_Hybrid:MX-NoLED
- removed Y1: 16Mhz, Crystal:Crystal_HC49-4H_Vertical, symbol Device:Crystal
- added Y1: Resonator, Crystal:Resonator-3Pin_W7.0mm_H2.5mm, symbol Device:Resonator
- Boot1: value Boot -> Boot1
- Reset1: value Reset -> Reset1
- renumbered C3 to C1, C4 to C2, C5 to C3, D17 to D16, D18 to D17, D19 to D18, D20 to D19, D21 to D20, D22 to D21, D23 to D22, D24 to D23, D25 to D24, D26 to D25, D27 to D26, D28 to D27, D29 to D28, D30 to D29, D31 to D30, D32 to D31, D33 to D32, D34 to D33, D35 to D34, D36 to D35, D37 to D36, D38 to D37, D39 to D38, D40 to D39, D41 to D40, D42 to D41, D43 to D42, D44 to D43, D45 to D44, D46 to D45, D47 to D46, D48 to D47, D49 to D48, D50 to D49, D51 to D50, D52 to D51, D53 to D52, D54 to D53, D55 to D54, D56 to D55, D57 to D56, D58 to D57, D59 to D58, D60 to D59, D61 to D60, D62 to D61, D63 to D62, D64 to D63, D65 to D64, D66 to D65, D67 to D66, D69 to D67, D70 to D68, D71 to D69, D72 to D70, D73 to D71, D74 to D72, D16 to D73, D75 to D74, D76 to D75, D77 to D76, D78 to D77, D79 to D78, D80 to D79, D81 to D80, J2 to J1, J1 to J2, D82 to LED1, MX15 to MX14, MX16 to MX15, MX17 to MX16, MX18 to MX17, MX19 to MX18, MX20 to MX19, MX21 to MX20, MX22 to MX21, MX23 to MX22, MX24 to MX23, MX25 to MX24, MX26 to MX25, MX27 to MX26, MX28 to MX27, MX29 to MX28, MX30 to MX29, MX31 to MX30, MX32 to MX31, MX33 to MX32, MX34 to MX33, MX35 to MX34, MX36 to MX35, MX37 to MX36, MX38 to MX37, MX39 to MX38, MX40 to MX39, MX41 to MX40, MX42 to MX41, MX43 to MX42, MX44 to MX43, MX45 to MX44, MX46 to MX45, MX47 to MX46, MX48 to MX47, MX49 to MX48, MX50 to MX49, MX51 to MX50, MX52 to MX51, MX53 to MX52, MX54 to MX53, MX55 to MX54, MX56 to MX55, MX57 to MX56, MX58 to MX57, MX59 to MX58, MX60 to MX59, MX61 to MX60, MX62 to MX61, MX63 to MX62, MX64 to MX63, MX65 to MX64, MX67 to MX65, MX68 to MX66, MX69 to MX67, MX70 to MX68, MX71 to MX69, MX72 to MX70, MX14 to MX71, MX73 to MX72, MX74 to MX73, MX75 to MX74, MX76 to MX75, MX77 to MX76, MX78 to MX77, MX79 to MX78, R5 to R4, R4 to R5
Connections:
- net D+: now also U1.16 (PD2); no longer U1.17 (PD3)
- net D-: now also U1.17 (PD3); no longer U1.16 (PD2)
- net GND: now also J1.6 (Shield), Y1.2
- net col5: now also U1.15 (PD1); no longer U1.20 (PD6)
- net at U1.12 (XTAL2): now also Y1.3
- net at U1.13 (XTAL1): now also Y1.1
Other:
- moved on the sheet: D10, D11, D12, D13, D14, D15, D16, D17, D18, D19, D20, D21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
